File: m68k.sch (KiCad schematic (older format))
At the start: 35 parts

Commit message: save
Parts:
- removed C? (x2): 100n, symbol C_Small
- removed J?: ISP, symbol CONN_02X03
- removed J?: UART, symbol CONN_01X03
- removed U?: 25LC_EEPROM, symbol 25LC_EEPROM
- removed U? (x2): AS6C4008, symbol AS6C4008
- removed U?: ATMEGA328P-AU, TQFP32, symbol ATMEGA328P-AU
- removed U?: LM1117-3.3, symbol LM1117-3.3
- added C? (x6): 100n, symbol C_Small
- added J?: Power, symbol CONN_01X04
- added R? (x2): 10k, symbol R_Small
- added SW?: SW_Push_Dual, symbol SW_Push_Dual
- added U? (x2): AT28BV64, symbol AT28BV64
- added U?: XO91-16, symbol XO91
- added U?: XO91-50, symbol XO91
- added U?: LM1084IT-3.3/NOPB, TO_SOT_Packages_THT:TO-220_Vertical, symbol LM1084IT-3.3/NOPB
- added U?: MCP23008, symbol MCP23008
- added U?: MCP23017, symbol MCP23017
- added U?: AS6C8016, symbol AS6C8016
Connections:
- net +3V3: now also J?.4 (P4), C?.1, C?.1, C?.2, C?.2, C?.2, C?.2, R?.2, R?.2, U?.18 (VCC), U?.18 (~RESET), U?.2 (OUT), U?.28 (VCC), U?.28 (VCC), U?.4 (VCC), U?.4 (VCC), U?.5 (A0), U?.6 (~RESET), U?.9 (VCC)
- net +5V: now also J?.2 (P2), J?.3 (P3), J?.4 (P4), U?.3 (IN)
- net A1: now also J?.5 (P5), U?.10 (A0), U?.10 (A0), U?.5 (A0)
- net A10: now also J?.14 (P14), U?.24 (A9), U?.24 (A9), U?.27 (A9)
- net A11: now also J?.15 (P15), U?.21 (A10), U?.21 (A10), U?.26 (A10)
- net A12: now also J?.16 (P16), U?.23 (A11), U?.23 (A11), U?.25 (A11)
- net A13: now also J?.17 (P17), U?.2 (A12), U?.2 (A12), U?.24 (A12)
- net A14: now also J?.18 (P18), U?.23 (A13)
- net A15: now also J?.19 (P19), U?.22 (A14)
- net A16: now also J?.20 (P20), U?.21 (A15)
- net A17: now also J?.21 (P21), U?.20 (A16)
- net A18: now also J?.22 (P22), U?.19 (A17)
- net A19: now also J?.23 (P23), U?.18 (A18)
- net A2: now also J?.6 (P6), U?.4 (A1), U?.9 (A1), U?.9 (A1)
- net A20: now also J?.24 (P24); no longer U?.39 (P39)
- net A21: now also J?.25 (P25); no longer U?.40 (P40)
- net A22: now also J?.26 (P26); no longer U?.41 (P41)
- net A23: now also J?.27 (P27); no longer U?.42 (P42)
- net A3: now also J?.7 (P7), U?.3 (A2), U?.8 (A2), U?.8 (A2)
- net A4: now also J?.8 (P8), U?.2 (A3), U?.7 (A3), U?.7 (A3)
- net A5: now also J?.9 (P9), U?.1 (A4), U?.6 (A4), U?.6 (A4)
- net A6: now also J?.10 (P10), U?.44 (A5), U?.5 (A5), U?.5 (A5)
- net A7: now also J?.11 (P11), U?.4 (A6), U?.4 (A6), U?.43 (A6)
- net A8: now also J?.12 (P12), U?.3 (A7), U?.3 (A7), U?.42 (A7)
- net A9: now also J?.13 (P13), U?.25 (A8), U?.25 (A8), U?.28 (A8)
- net AS_N: now also U?.6 (P6)
- net AVEC_N: now also J?.50 (P50)
- net BERR_N: now also U?.12 (P12); no longer U?.12 (BERR), U?.38 (P38)
- net BG_N: now also J?.49 (P49)
- net BOOT: now also U?.20 (P20), U?.10 (GPB0); no longer U?.36 (GTS1)
- net BR_N: now also J?.48 (P48)
- net CLK_16MHz: now also U?.3 (OUT)
- net D0: now also J?.28 (P28), U?.1 (GPB0), U?.11 (IO0); no longer U?.2 (P2)
- net D1: now also J?.29 (P29), U?.12 (IO1), U?.2 (GPB1); no longer U?.3 (P3)
- net D10: now also J?.38 (P38), U?.13 (IO2), U?.23 (GPA2); no longer U?.18 (P18)
- net D11: now also J?.39 (P39), U?.15 (IO3), U?.24 (GPA3); no longer U?.19 (P19)
- net D12: now also J?.40 (P40), U?.16 (IO4), U?.25 (GPA4); no longer U?.20 (P20)
- net D13: now also J?.41 (P41), U?.17 (IO5), U?.26 (GPA5); no longer U?.21 (P21)
- net D14: now also J?.42 (P42), U?.18 (IO6), U?.27 (GPA6); no longer U?.22 (P22)
- net D15: now also J?.43 (P43), U?.19 (IO7), U?.28 (GPA7); no longer U?.23 (P23)
- net D2: now also J?.30 (P30), U?.13 (IO2), U?.3 (GPB2); no longer U?.5 (P5)
- net D3: now also J?.31 (P31), U?.15 (IO3), U?.4 (GPB3); no longer U?.6 (P6)
- net D4: now also J?.32 (P32), U?.16 (IO4), U?.5 (GPB4); no longer U?.7 (P7)
- net D5: now also J?.33 (P33), U?.17 (IO5), U?.6 (GPB5); no longer U?.8 (P8)
- net D6: now also J?.34 (P34), U?.18 (IO6), U?.7 (GPB6); no longer U?.12 (P12)
- net D7: now also J?.35 (P35), U?.19 (IO7), U?.8 (GPB7); no longer U?.13 (P13)
- net D8: now also J?.36 (P36), U?.11 (IO0), U?.21 (GPA0); no longer U?.14 (P14)
- net D9: now also J?.37 (P37), U?.12 (IO1), U?.22 (GPA1); no longer U?.16 (P16)
- net DTACK_N: now also J?.44 (P44), U?.2 (P2); no longer U?.34 (GTS2)
- net GND: now also J?.1 (P1), J?.3 (P3), C?.1, C?.1, C?.1, C?.1, C?.2, C?.2, J?.1 (P1), J?.2 (P2), SW?.1, SW?.3, U?.1 (GND), U?.10 (GND), U?.14 (GND), U?.14 (GND), U?.15 (A0), U?.16 (A1), U?.17 (A2), U?.2 (GND), U?.2 (GND), U?.3 (A2), U?.4 (A1), U?.9 (GND)
- net HALT_N: now also SW?.4; no longer U?.9 (HALT)
- net LDS_N: now also J?.46 (P46), U?.7 (P7); no longer U?.29 (P29)
- net OE_N: now also U?.5 (P5), U?.22 (OE), U?.22 (OE); no longer U?.28 (P28)
- net R/W: now also J?.45 (P45), U?.3 (P3), U?.27 (WE), U?.27 (WE); no longer U?.27 (P27)
- net RAM_LDS_N: now also U?.13 (P13); no longer U?.32 (P32)
- net RAM_UDS_N: now also U?.14 (P14); no longer U?.37 (P37)
- net RESET_N: now also SW?.2; no longer U?.10 (RESET)
- net UDS_N: now also J?.47 (P47), U?.8 (P8); no longer U?.30 (P30)
- net CLK_AVR renamed CLK_FROM_CPLD
- net CLK_FROM_CPLD: now also U?.19 (P19)
- net CLK_CPLD renamed CLK_50MHz
- net CLK_50MHz: now also U?.3 (OUT)
- net DCLK: no longer names the net of U?.44 (GCK2)
- net DIN: no longer names the net of U?.31 (P31)
- new net: R?.1, U?.1 (EN) (x2)
- new net DTACK_TRIG: U?.11 (GPB1), U?.21 (P21)
- new net EEPROM_LDS_N: U?.16 (P16), U?.20 (CE)
- new net EEPROM_UDS_N: U?.18 (P18), U?.20 (CE)
- new net R/~W: U?.17 (~WE)
- new net SCL: U?.1 (SCL), U?.12 (SCL)
- new net SDA: U?.13 (SDA), U?.2 (SDA)
- new net ~BERR: U?.12 (BERR)
- new net ~HALT: U?.9 (HALT)
- new net ~LDS: U?.39 (~LB)
- new net ~OE: U?.41 (~OE)
- new net ~RAM_CE: U?.6 (~CE)
- new net ~RESET: U?.10 (RESET)
- new net ~UDS: U?.40 (~UB)
Other:
- note added: "Längeres DTACK für eeprom."
- note added: "OE_N = 1 wenn BOOT=1, sonst Buskollision"
- note added: "i2c-addr: 0x20"
- note added: "i2c-addr: 0x21"
- moved on the sheet: C?, J?, U?

Commit message: further work
Parts:
- removed C?: 100n, symbol C_Small
- removed J?: CONN_02X25, symbol CONN_02X25
- removed R? (x10): 10k, symbol R_Small
- added C4: 100n, Capacitors_SMD:C_0805_HandSoldering, symbol C_Small
- added J4: CONN_02X30, Connectors:IDC_Header_Straight_60pins, symbol CONN_02X30
- added J5: I2C, Pin_Headers:Pin_Header_Straight_1x03_Pitch2.54mm, symbol CONN_01X03
- added R15, R16: 2k, Resistors_SMD:R_0805_HandSoldering, symbol R_Small
- added RN1: R_Network10, Resistors_THT:R_Array_SIP11, symbol R_Network10
- C1, C10, C11, C12, C13, C14, C15, C16, C2, C3, C6, C7, C8, C9: renamed from C?; footprint (none) -> Capacitors_SMD:C_0805_HandSoldering
- J1: renamed from J?; footprint (none) -> Pin_Headers:Pin_Header_Straight_1x04_Pitch2.54mm
- J2: renamed from J?; footprint (none) -> Pin_Headers:Pin_Header_Straight_1x03_Pitch2.54mm
- J3: renamed from J?; footprint (none) -> Pin_Headers:Pin_Header_Straight_1x06_Pitch2.54mm
- R13, R14, R3, R4: renamed from R?; footprint (none) -> Resistors_SMD:R_0805_HandSoldering
- SW1: renamed from SW?; footprint (none) -> Buttons_Switches_THT:SW_TH_Tactile_Omron_B3F-10xx
- U1: renamed from U?; footprint (none) -> Housings_QFP:TQFP-64_14x14mm_Pitch0.8mm
- U10: renamed from U?; footprint (none) -> Housings_SOIC:SOIC-18W_7.5x11.6mm_Pitch1.27mm
- U2: renamed from U?; footprint (none) -> Housings_SSOP:TSSOP-44_4.4x11.2mm_Pitch0.5mm
- U4, U5, U7: renamed from U?; footprint (none) -> SMD_Packages:SOIC-28
- U6: renamed from U?; footprint (none) -> Housings_QFP:TQFP-44_10x10mm_Pitch0.8mm
- U8, U9: renamed from U?; footprint (none) -> Crystals:Crystal_SMD_EuroQuartz_MQ-4pin_7.0x5.0mm_HandSoldering
- gave numbers to parts that had none: 1
Connections:
- net BERR_N is gone; now on net ~BERR: U6.12 (P12)
- net HALT_N is gone; now on net ~HALT: SW1.4
- net LDS_N is gone; now on net ~LDS: U1.64 (LDS), U6.7 (P7)
- net OE_N is gone; now on net ~OE: U4.22 (OE), U5.22 (OE), U6.5 (P5)
- net R/W is gone; now on net R/~W: R4.2, U4.27 (WE), U5.27 (WE), U6.3 (P3)
- net RAM_LDS_N is gone; now on net ~RAM_CE: U6.13 (P13)
- net RAM_UDS_N is gone; now on net ~EEPROM_LDS: U6.14 (P14)
- net RESET_N is gone; now on net ~RESET: SW1.2
- net UDS_N is gone; now on net ~UDS: U1.63 (UDS), U6.8 (P8)
- net +3V3: now also C10.2, C11.2, C12.2, U2.11 (VCC), U2.33 (VCC), U6.15 (VCCINT), U6.26 (VCCIO), U6.35 (VCCINT), C4.1, J4.4 (P4), R15.1, R16.1, RN1.1 (common)
- net +5V: now also J4.2 (P2)
- net A1: now also J4.5 (P5)
- net A10: now also J4.14 (P14)
- net A11: now also J4.15 (P15)
- net A12: now also J4.16 (P16)
- net A13: now also U6.23 (P23), J4.17 (P17)
- net A14: now also U6.27 (P27), J4.18 (P18)
- net A15: now also U6.28 (P28), J4.19 (P19)
- net A16: now also U6.29 (P29), J4.20 (P20)
- net A17: now also U6.30 (P30), J4.21 (P21)
- net A18: now also U6.31 (P31), J4.22 (P22)
- net A19: now also U6.32 (P32), J4.23 (P23)
- net A2: now also J4.6 (P6)
- net A20: now also U6.37 (P37), J4.24 (P24)
- net A21: now also U6.38 (P38), J4.25 (P25)
- net A22: now also U6.39 (P39), J4.26 (P26)
- net A23: now also U6.40 (P40), J4.27 (P27)
- net A3: now also J4.7 (P7)
- net A4: now also J4.8 (P8)
- net A5: now also J4.9 (P9)
- net A6: now also J4.10 (P10)
- net A7: now also J4.11 (P11)
- net A8: now also J4.12 (P12)
- net A9: now also J4.13 (P13)
- net BOOT: now also U6.19 (P19), J4.54 (P54); no longer U6.20 (P20)
- net CLK_16MHz: now also U6.1 (GCK3)
- net CLK_FROM_CPLD: now also U6.18 (P18); no longer U6.19 (P19)
- net D0: now also U2.7 (DQ0), J4.28 (P28)
- net D1: now also U2.8 (DQ1), J4.29 (P29)
- net D10: now also U2.31 (DQ10), J4.38 (P38)
- net D11: now also U2.32 (DQ11), J4.39 (P39)
- net D12: now also U2.35 (DQ12), J4.40 (P40)
- net D13: now also U2.36 (DQ13), J4.41 (P41)
- net D14: now also U2.37 (DQ14), J4.42 (P42)
- net D15: now also U2.38 (DQ15), J4.43 (P43)
- net D2: now also U2.9 (DQ2), J4.30 (P30)
- net D3: now also U2.10 (DQ3), J4.31 (P31)
- net D4: now also U2.13 (DQ4), J4.32 (P32)
- net D5: now also U2.14 (DQ5), J4.33 (P33)
- net D6: now also U2.15 (DQ6), J4.34 (P34)
- net D7: now also U2.16 (DQ7), J4.35 (P35)
- net D8: now also U2.29 (DQ8), J4.36 (P36)
- net D9: now also U2.30 (DQ9), J4.37 (P37)
- net DTACK_TRIG: now also U6.20 (P20); no longer U6.21 (P21)
- net GND: now also U1.56 (GND), U1.7 (GND), U2.12 (VSS), U2.34 (VSS), C4.2, J4.1 (P1), J4.3 (P3), J5.1 (P1)
- net R/~W: now also J4.45 (P45)
- net SCL: now also J5.3 (P3), R15.2
- net SDA: now also J5.2 (P2), R16.2
- net ~BERR: now also RN1.7 (R6)
- net ~HALT: now also RN1.9 (R8)
- net ~LDS: now also J4.46 (P46)
- net ~RESET: now also RN1.8 (R7)
- net ~UDS: now also J4.47 (P47)
- net A0: no longer names the net of U1.19 (A0)
- net AS_N renamed ~AS
- net AVEC_N renamed ~AVEC
- net ~AVEC: now also J4.50 (P50), RN1.3 (R2)
- net BG_N renamed ~BG
- net ~BG: now also J4.49 (P49), RN1.11 (R10)
- net BR_N renamed ~BR
- net ~BR: now also J4.48 (P48), RN1.10 (R9)
- net DTACK_N renamed ~DTACK
- net ~DTACK: now also J4.44 (P44), RN1.2 (R1)
- net EEPROM_LDS_N renamed ~EEPROM_LDS
- net ~EEPROM_LDS: no longer U6.16 (P16)
- net EEPROM_UDS_N renamed ~EEPROM_UDS
- net ~EEPROM_UDS: now also U6.16 (P16); no longer U6.18 (P18)
- net FC0: no longer names the net of U1.18 (FC0)
- net FC1: no longer names the net of U1.17 (FC1)
- net FC2: no longer names the net of U1.16 (FC2)
- net IPL0_N renamed ~IPL0
- net ~IPL0: now also J4.51 (P51), RN1.6 (R5)
- net IPL1_N renamed ~IPL1
- net ~IPL1: now also J4.52 (P52), RN1.5 (R4)
- net IPL2_N renamed ~IPL2
- net ~IPL2: now also J4.53 (P53), RN1.4 (R3)
- no-connect marks 0 -> 27
Other:
- note added: "#OE = 1 wenn BOOT=1, sonst Buskollision"
- note removed: "OE_N = 1 wenn BOOT=1, sonst Buskollision"
- moved on the sheet: C10, C11, C12, C13, C14, C15, C16, C3, C6, C7, J1, J3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

Commit message: further improvements
Parts:
- added D1: LED, LEDs:LED_0805, symbol LED
- added J?: CONN_01X06, symbol CONN_01X06
- added J?: CONN_01X03, symbol CONN_01X03
- added R1: 750, Resistors_SMD:R_0805_HandSoldering, symbol R_Small
- U2: footprint Housings_SSOP:TSSOP-44_4.4x11.2mm_Pitch0.5mm -> custom:TSOP44
Connections:
- net +3V3: now also R1.1
- net A13: now also U6.21 (P21); no longer U6.23 (P23)
- net A14: now also U6.22 (P22); no longer U6.27 (P27)
- net A15: now also U6.23 (P23); no longer U6.28 (P28)
- net A16: now also U6.27 (P27); no longer U6.29 (P29)
- net A17: now also U6.28 (P28); no longer U6.30 (P30)
- net A18: now also U6.29 (P29); no longer U6.31 (P31)
- net A19: now also U6.30 (P30); no longer U6.32 (P32)
- net A20: now also U6.31 (P31); no longer U6.37 (P37)
- net A21: now also U6.32 (P32); no longer U6.38 (P38)
- net A22: now also U6.37 (P37); no longer U6.39 (P39)
- net A23: now also U6.38 (P38); no longer U6.40 (P40)
- net GND: now also D1.1 (K)
- net at U6.33 (GSR): now also J?.1 (P1)
- net at U6.34 (GTS2): now also J?.2 (P2)
- net at U6.36 (GTS1): now also J?.3 (P3)
- net CS2: now reaches U6.41 (P41)
- net CS2: now also J4.57 (P57)
- net CS3: now reaches U6.42 (P42)
- net CS3: now also J4.58 (P58)
- net at U10.12 (GPB2): now also J?.6 (P6)
- net at U10.13 (GPB3): now also J?.5 (P5)
- net at U10.14 (GPB4): now also J?.4 (P4)
- net at U10.15 (GPB5): now also J?.3 (P3)
- net at U10.16 (GPB6): now also J?.2 (P2)
- net at U10.17 (GPB7): now also J?.1 (P1)
- net CS0: now reaches J4.55 (P55)
- net CS0: now also U6.39 (P39)
- net CS1: now reaches J4.56 (P56)
- net CS1: now also U6.40 (P40)
- new net: D1.2 (A), R1.2
- no-connect marks 27 -> 10
Changed lines of the file:
@@
-$EndComp
-$Comp
-L XC9572XL-VQ44 U6
-U 1 1 59881A68
-P 10350 2650
-F 0 "U6" H 10550 4100 60  0000 C CNN
-F 1 "XC9572XL-VQ44" H 10300 1150 60  0000 C CNN
-F 2 "Housings_QFP:TQFP-44_10x10mm_Pitch0.8mm" H 10300 2250 60  0001 C CNN
-F 3 "" H 10300 2250 60  0001 C CNN
-	1    10350 2650
-	1    0    0    -1
 $EndComp
 $Comp
@@
 Text Label 9550 2550 2    60   ~ 0
 TMS
-Text Label 10850 3550 0    60   ~ 0
+Text Label 10850 3350 0    60   ~ 0
 A20
-Text Label 10850 3650 0    60   ~ 0
+Text Label 10850 3450 0    60   ~ 0
 A21
 Text Label 10850 1950 0    60   ~ 0
@@
 Text Label 10850 1450 0    60   ~ 0
 R/~W
-Text Label 10850 3750 0    60   ~ 0
+Text Label 10850 3550 0    60   ~ 0
 A22
-Text Label 10850 3850 0    60   ~ 0
+Text Label 10850 3650 0    60   ~ 0
 A23
 Text Label 4700 3400 2    60   ~ 0
@@
 Text Label 10050 6000 2    60   ~ 0
 A23
+Text Label 10850 2650 0    60   ~ 0
+A13
+Text Label 10850 2750 0    60   ~ 0
+A14
 Text Label 10850 2850 0    60   ~ 0
-A13
+A15
 Text Label 10850 2950 0    60   ~ 0
-A14
+A16
 Text Label 10850 3050 0    60   ~ 0
-A15
+A17
 Text Label 10850 3150 0    60   ~ 0
-A16
+A18
 Text Label 10850 3250 0    60   ~ 0
-A17
-Text Label 10850 3350 0    60   ~ 0
-A18
-Text Label 10850 3450 0    60   ~ 0
 A19
 Text Label 10850 2450 0    60   ~ 0
@@
 F 0 "U2" H 5250 3450 60  0000 C CNN
 F 1 "AS6C8016" H 5150 900 60  0000 C CNN
-F 2 "Housings_SSOP:TSSOP-44_4.4x11.2mm_Pitch0.5mm" H 5150 2350 60  0001 C CNN
+F 2 "custom:TSOP44" H 5150 2350 60  0001 C CNN
 F 3 "" H 5150 2350 60  0001 C CNN
 	1    5150 2350
@@
 	1    0    0    -1
 $EndComp
-NoConn ~ 12500 2650
-NoConn ~ 12500 2750
-NoConn ~ 12500 2850
-NoConn ~ 12500 2950
-NoConn ~ 12500 3050
-NoConn ~ 12500 3150
 NoConn ~ 13500 2450
 NoConn ~ 13500 4650
@@
 	2200 6800 2550 6800
 NoConn ~ 9750 1450
-NoConn ~ 9750 1650
-NoConn ~ 9750 1750
-NoConn ~ 9750 1850
-NoConn ~ 10850 2650
-NoConn ~ 10850 2750
-NoConn ~ 10850 3950
-NoConn ~ 10850 4050
 Connection ~ 9750 3500
 Connection ~ 9750 3450
@@
 	1    0    0    -1
 $EndComp
-NoConn ~ 10050 7400
-NoConn ~ 10050 7500
 NoConn ~ 10050 7600
-NoConn ~ 10550 7400
-NoConn ~ 10550 7500
 NoConn ~ 10550 7600
 $Comp
@@
 Wire Notes Line
 	11950 6300 11950 1750
+$Comp
+L LED D1
+U 1 1 598F0960
+P 6350 5400
+F 0 "D1" H 6350 5500 50  0000 C CNN
+F 1 "LED" H 6350 5300 50  0000 C CNN
+F 2 "LEDs:LED_0805" H 6350 5400 50  0001 C CNN
+F 3 "" H 6350 5400 50  0001 C CNN
+	1    6350 5400
+	0    -1   -1   0
+$EndComp
+$Comp
+L R_Small R1
+U 1 1 598F0A1F
+P 6350 5150
+F 0 "R1" H 6380 5170 50  0000 L CNN
+F 1 "750" H 6380 5110 50  0000 L CNN
+F 2 "Resistors_SMD:R_0805_HandSoldering" H 6350 5150 50  0001 C CNN
+F 3 "" H 6350 5150 50  0001 C CNN
+	1    6350 5150
+	1    0    0    -1
+$EndComp
+$Comp
+L GND #PWR034
+U 1 1 598F0AC4
+P 6350 5550
+F 0 "#PWR034" H 6350 5300 50  0001 C CNN
+F 1 "GND" H 6350 5400 50  0000 C CNN
+F 2 "" H 6350 5550 50  0001 C CNN
+F 3 "" H 6350 5550 50  0001 C CNN
+	1    6350 5550
+	1    0    0    -1
+$EndComp
+$Comp
+L +3V3 #PWR035
+U 1 1 598F0C18
+P 6350 5050
+F 0 "#PWR035" H 6350 4900 50  0001 C CNN
+F 1 "+3V3" H 6350 5190 50  0000 C CNN
+F 2 "" H 6350 5050 50  0001 C CNN
+F 3 "" H 6350 5050 50  0001 C CNN
+	1    6350 5050
+	1    0    0    -1
+$EndComp
+$Comp
+L CONN_01X06 J?
+U 1 1 598F1D1B
+P 12300 2900
+F 0 "J?" H 12300 3250 50  0000 C CNN
+F 1 "CONN_01X06" V 12400 2900 50  0000 C CNN
+F 2 "" H 12300 2900 50  0001 C CNN
+F 3 "" H 12300 2900 50  0001 C CNN
+	1    12300 2900
+	-1   0    0    1
+$EndComp
+$Comp
+L XC9572XL-VQ44 U6
+U 1 1 59881A68
+P 10350 2650
+F 0 "U6" H 10550 4100 60  0000 C CNN
+F 1 "XC9572XL-VQ44" H 10300 1150 60  0000 C CNN
+F 2 "Housings_QFP:TQFP-44_10x10mm_Pitch0.8mm" H 10300 2250 60  0001 C CNN
+F 3 "" H 10300 2250 60  0001 C CNN
+	1    10350 2650
+	1    0    0    -1
+$EndComp
+$Comp
+L CONN_01X03 J?
+U 1 1 598F47DA
+P 9550 1750
+F 0 "J?" H 9550 1950 50  0000 C CNN
+F 1 "CONN_01X03" V 9650 1750 50  0000 C CNN
+F 2 "" H 9550 1750 50  0001 C CNN
+F 3 "" H 9550 1750 50  0001 C CNN
+	1    9550 1750
+	-1   0    0    1
+$EndComp
+Text Label 10850 3750 0    60   ~ 0
+CS0
+Text Label 10850 3850 0    60   ~ 0
+CS1
+Text Label 10850 3950 0    60   ~ 0
+CS2
+Text Label 10850 4050 0    60   ~ 0
+CS3
+Text Label 10050 7400 2    60   ~ 0
+CS0
+Text Label 10050 7500 2    60   ~ 0
+CS2
+Text Label 10550 7400 0    60   ~ 0
+CS1
+Text Label 10550 7500 0    60   ~ 0
+CS3
 $EndSCHEMATC
