File: schematic/m68k.kicad_pcb (KiCad board)
At the start: 2 copper layers, 45 parts, among them J1 Power, J2 CONN_01X03, J3 JTAG, J4 CONN_02X30, J5 I2C, J6 CONN_02X30, J7 CONN_01X02, J8 CONN_02X30, J9 CONN_01X03, SW1 SW_Push_Dual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

Commit message: routing started
Routing:
- net /A11: track 0.00 -> 93.7 mm, vias 0 -> 2
- net /A21: track 0.00 -> 91.5 mm, vias 0 -> 2
- net /A23: track 0.00 -> 91.4 mm, vias 0 -> 2
- net /A13: track 0.00 -> 91.2 mm, vias 0 -> 2
- net /A15: track 0.00 -> 91.2 mm, vias 0 -> 2
- net /A17: track 0.00 -> 91.0 mm, vias 0 -> 2
- net /A19: track 0.00 -> 90.9 mm, vias 0 -> 2
- net /A12: track 0.00 -> 89.1 mm, vias 0 -> 2
- net /A22: track 0.00 -> 88.5 mm, vias 0 -> 2
- net /A16: track 0.00 -> 88.2 mm, vias 0 -> 2
- net /A18: track 0.00 -> 88.0 mm, vias 0 -> 2
- net /A20: track 0.00 -> 87.8 mm, vias 0 -> 2
- net /A14: track 0.00 -> 87.7 mm, vias 0 -> 2
- net +3V3: track 0.00 -> 6.90 mm
Other:
- net class Power: clearance 0.2 -> 0.15

Commit message: weiter
Routing:
- net /A1: track 0.00 -> 156.9 mm, vias 0 -> 6
- net /A3: track 0.00 -> 153.8 mm, vias 0 -> 6
- net /A2: track 0.00 -> 152.5 mm, vias 0 -> 6
- net /A5: track 0.00 -> 149.8 mm, vias 0 -> 6
- net /A4: track 0.00 -> 148.4 mm, vias 0 -> 6
- net /A7: track 0.00 -> 141.5 mm, vias 0 -> 6
- net /A6: track 0.00 -> 141.5 mm, vias 0 -> 6
- net /A8: track 0.00 -> 135.5 mm, vias 0 -> 6
- net /A9: track 0.00 -> 114.7 mm, vias 0 -> 4
- net /A10: track 0.00 -> 109.1 mm, vias 0 -> 4
- net /A13: track 91.2 -> 113.7 mm, vias 2 -> 6
- net /A19: track 90.9 -> 109.2 mm
- net /A18: track 88.0 -> 105.7 mm
- net /A17: track 91.0 -> 108.1 mm
- net /A16: track 88.2 -> 104.7 mm
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
Commit message: weiter
Parts:
- moved C13 10.5 mm to (84.3, 63.5)
- moved R13 10.5 mm to (84.4, 59.6)
- moved U8 10.5 mm to (74.5, 61.0)
- moved R2 2.49 mm to (125.9, 108.7)
- moved C8 1.57 mm to (145.1, 63.1), turned to 180 degrees
- moved C10 1.32 mm to (121.9, 114.5)
- moved C11 1.27 mm to (113.8, 103.2)
- moved U4 0.05 mm to (157.7, 66.6)
Routing:
- net /D15: track 0.00 -> 194.1 mm, vias 0 -> 8
- net /D14: track 0.00 -> 192.0 mm, vias 0 -> 8
- net /D10: track 0.00 -> 189.9 mm, vias 0 -> 9
- net /D8: track 0.00 -> 188.8 mm, vias 0 -> 10
- net /D9: track 0.00 -> 187.6 mm, vias 0 -> 9
- net /D0: track 0.00 -> 185.8 mm, vias 0 -> 7
- net /D11: track 0.00 -> 185.0 mm, vias 0 -> 9
- net /D12: track 0.00 -> 184.2 mm, vias 0 -> 8
- net /D13: track 0.00 -> 183.6 mm, vias 0 -> 8
- net /D1: track 0.00 -> 178.8 mm, vias 0 -> 7
- net /D2: track 0.00 -> 176.5 mm, vias 0 -> 7
- net /D4: track 0.00 -> 173.8 mm, vias 0 -> 8
- net /D3: track 0.00 -> 170.9 mm, vias 0 -> 8
- net /D5: track 0.00 -> 169.2 mm, vias 0 -> 8
- net /D6: track 0.00 -> 168.7 mm, vias 0 -> 8
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
Commit message: weiter
Parts:
- moved C13 14.9 mm to (75.4, 51.6), turned to 0 degrees
- moved R13 9.64 mm to (75.4, 56.3), turned to 0 degrees
- moved C4 4.85 mm to (117.3, 75.3)
- moved U8 4.06 mm to (75.3, 65.0), turned to 270 degrees
- moved R4 3.39 mm to (87.4, 65.9), turned to 90 degrees
- moved J5 2.49 mm to (86.8, 47.0)
- moved C9 0.82 mm to (146.9, 78.3)
Routing:
- net /~BG: track 37.1 -> 161.5 mm, vias 2 -> 5
- net /~BR: track 34.1 -> 133.4 mm, vias 1 -> 3
- net /~EEPROM_LDS: track 0.00 -> 93.7 mm, vias 0 -> 2
- net /~DTACK: track 80.8 -> 174.0 mm, vias 0 -> 6
- net /~EEPROM_UDS: track 0.00 -> 81.3 mm, vias 0 -> 2
- net /~LDS: track 58.5 -> 124.9 mm, vias 2 -> 6
- net /~AVEC: track 33.5 -> 98.9 mm
- net /~UDS: track 61.9 -> 126.1 mm, vias 2 -> 6
- net /R/~W: track 157.7 -> 218.3 mm, vias 7 -> 9
- net /~AS: track 0.00 -> 53.3 mm, vias 0 -> 2
- net /~RAM_CE: track 0.00 -> 49.5 mm, vias 0 -> 2
- net +3V3: track 98.4 -> 120.9 mm
- net /CLK_68k: track 0.00 -> 10.9 mm
- net /CLK_50MHz: track 0.00 -> 10.3 mm
- net Net-(R4-Pad1): track 0.00 -> 8.30 mm
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
Commit message: weiter
Parts:
- moved R2 10.7 mm to (116.7, 103.3), turned to 90 degrees
- moved J7 10.5 mm to (131.5, 116.9)
- moved C16 3.34 mm to (142.3, 119.0)
- moved J3 3.07 mm to (101.7, 123.1)
- moved U10 2.90 mm to (147.2, 109.8)
- moved J9 2.72 mm to (147.1, 119.9)
- moved R3 1.82 mm to (82.2, 80.7), turned to 180 degrees
- moved C12 0.99 mm to (109.0, 124.7)
Routing:
- net /~IPL0: track 36.1 -> 183.2 mm, vias 2 -> 5
- net /~IPL1: track 32.3 -> 178.0 mm, vias 2 -> 5
- net /~IPL2: track 34.6 -> 178.9 mm, vias 2 -> 5
- net /SCL: track 0.00 -> 122.6 mm, vias 0 -> 2
- net /SDA: track 0.00 -> 120.1 mm, vias 0 -> 2
- net /~RESET: track 0.00 -> 119.3 mm, vias 0 -> 5
- net /~HALT: track 0.00 -> 102.7 mm, vias 0 -> 5
- net /~OE: track 36.5 -> 131.0 mm, vias 3 -> 7
- net /CS0: track 81.0 -> 163.0 mm, vias 1 -> 4
- net /CS1: track 78.7 -> 157.8 mm, vias 1 -> 4
- net /CS2: track 82.5 -> 158.5 mm, vias 1 -> 4
- net /CS3: track 80.4 -> 153.8 mm, vias 1 -> 4
- net /~AVEC: track 98.9 -> 169.4 mm, vias 2 -> 5
- net /CLK_FROM_CPLD: track 0.00 -> 68.4 mm, vias 0 -> 3
- net /CLK_16MHz: track 8.11 -> 67.1 mm, vias 0 -> 3
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
Commit message: routing done
Parts:
- moved C14 13.9 mm to (79.3, 114.1), turned to 0 degrees
- moved C7 11.1 mm to (121.0, 35.0), turned to 90 degrees
- moved U3 3.55 mm to (128.0, 33.7)
- moved U8 2.34 mm to (74.8, 62.7)
- moved C13 2.34 mm to (74.9, 49.3)
- moved C15 2.34 mm to (92.3, 39.3)
- moved C16 2.34 mm to (141.8, 116.8)
- moved C2 2.34 mm to (110.5, 78.7)
- moved C4 2.34 mm to (116.8, 73.0)
- moved J1 2.34 mm to (76.4, 34.0)
- moved J4 2.34 mm to (236.1, 116.0)
- moved J6 2.34 mm to (185.5, 116.0)
- moved J7 2.34 mm to (131.0, 114.6)
- moved J8 2.34 mm to (210.9, 116.0)
- moved J9 2.34 mm to (146.6, 117.6)
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Routing:
- net +3V3: track 146.6 -> 601.7 mm, vias 1 -> 5
- net GND: track 0.00 -> 197.9 mm, vias 0 -> 111
- net +5V: track 87.1 -> 267.4 mm, vias 1 -> 2
- net /A5: track 162.5 -> 259.4 mm
- net /A2: track 168.8 -> 263.0 mm
- net /A1: track 174.4 -> 266.4 mm
- net /A13: track 154.0 -> 238.0 mm
- net /A14: track 123.3 -> 206.7 mm
- net /A6: track 156.6 -> 231.8 mm
- net /A7: track 156.6 -> 228.9 mm
- net /A8: track 150.6 -> 222.2 mm
- net /D2: track 176.5 -> 246.0 mm
- net /D5: track 169.2 -> 238.3 mm
- net /A3: track 168.9 -> 237.1 mm
- net /A4: track 162.3 -> 228.2 mm
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- added copper zone on B.Cu, net GND
- added copper zone on F.Cu, net GND
Other:
- board outline added: 176.1 x 104 mm

Commit message: bla
Parts:
- U4, U5, U7: footprint SMD_Packages:SOIC-28 -> Housings_SOIC:SOIC-28W_7.5x17.9mm_Pitch1.27mm
- moved J1 37.1 mm to (113.3, 38.2), turned to 180 degrees
- moved R16 11.2 mm to (80.4, 40.7), turned to 0 degrees
- moved C6 8.75 mm to (123.8, 41.6)
- moved R15 7.12 mm to (80.4, 38.0), turned to 0 degrees
- moved C15 4.59 mm to (89.6, 35.6), turned to 270 degrees
- moved C7 4.27 mm to (124.4, 37.5)
- moved U7 3.93 mm to (98.3, 35.0), turned to 0 degrees
- moved C8 3.31 mm to (144.8, 57.5)
- moved R1 3.28 mm to (157.3, 38.6)
- moved U3 3.28 mm to (129.7, 36.6)
- moved D1 3.28 mm to (160.6, 38.5)
- moved U4 2.36 mm to (157.2, 62.0), turned to 90 degrees
- moved U5 2.18 mm to (157.2, 76.0), turned to 90 degrees
- moved J5 1.72 mm to (85.6, 43.1)
Routing:
- net +3V3: track 601.7 -> 419.8 mm, vias 5 -> 1
- net /SDA: track 147.1 -> 16.8 mm, vias 2 -> 1
- net +5V: track 267.4 -> 142.5 mm, vias 2 -> 1
- net /SCL: track 139.9 -> 17.1 mm, vias 2 -> 1
- net /~UDS: track 235.5 -> 176.0 mm, vias 8 -> 5
- net /~LDS: track 234.3 -> 175.0 mm, vias 8 -> 5
- net /A13: track 238.0 -> 193.4 mm, vias 10 -> 9
- net /A5: track 259.4 -> 216.9 mm
- net /A2: track 263.0 -> 223.1 mm
- net /A1: track 266.4 -> 228.7 mm
- net GND: track 197.9 -> 161.6 mm, vias 111 -> 83
- net /A14: track 206.7 -> 175.8 mm
- net /A6: track 231.8 -> 211.0 mm
- net /D6: track 221.5 -> 242.0 mm, vias 8 -> 9
- net /~OE: track 131.6 -> 111.1 mm, vias 7 -> 6
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
Commit message: bla
Parts:
- J1: value Power -> CONN_02X03; footprint Pin_Headers:Pin_Header_Straight_1x04_Pitch2.54mm -> Connectors:IDC_Header_Straight_6pins
- moved U3 19.2 mm to (148.3, 32.2)
- moved C7 19.2 mm to (143.1, 33.2)
- moved C6 19.2 mm to (142.4, 37.3)
- moved R1 18.6 mm to (139.6, 33.0), turned to 90 degrees
- moved D1 18.6 mm to (142.2, 41.1), turned to 180 degrees
- moved J1 17.1 mm to (129.8, 33.7)
- moved C9 3.43 mm to (146.2, 72.6)
Connections:
- J1 pad 2: GND -> +5V
- J1 pad 3: +5V -> GND
Routing:
- net /SCL: track 17.1 -> 141.4 mm, vias 1 -> 2
- net +3V3: track 419.8 -> 543.9 mm, vias 1 -> 4
- net /SDA: track 16.8 -> 138.2 mm, vias 1 -> 2
- net /~UDS: track 176.0 -> 226.8 mm, vias 5 -> 6
- net /~LDS: track 175.0 -> 223.3 mm, vias 5 -> 6
- net +5V: track 142.5 -> 189.1 mm, vias 1 -> 2
- net /A1: track 228.7 -> 261.6 mm
- net /A5: track 216.9 -> 247.0 mm
- net /~OE: track 111.1 -> 134.3 mm, vias 6 -> 7
- net /A12: track 190.8 -> 211.4 mm
- net /A8: track 205.2 -> 224.2 mm
- net /A6: track 211.0 -> 228.0 mm
- net /A13: track 193.4 -> 209.7 mm
- net Net-(D1-Pad2): track 0.00 -> 15.7 mm, vias 0 -> 2
- net /A4: track 216.8 -> 230.0 mm
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