File: schematic/extboard/extboard.sch (KiCad schematic (older format))
At the start: 1 part

Commit message: Entwurf extboard
Parts:
- added C?: 10n, symbol C_Small
- added C? (x4): 100n, symbol C_Small
- added J?: USB_B, symbol USB_B
- added J?: SD_Card, 10067847-001, symbol SD_Card
- added J?: Conn_01x02, symbol Conn_01x02
- added L?: L_Small, symbol L_Small
- added Q?: Q_NPN_BEC, symbol Q_NPN_BEC
- added R?: 33k, symbol R_Small
- added R? (x2): 150, symbol R_Small
- added R? (x2): 10k, symbol R_Small
- added U?: SST26VF, symbol SST26VF
- added U?: P8X32A, symbol P8X32A
- added U?: 24LC512, Housings_SOIC:SOIC-8_3.9x4.9mm_Pitch1.27mm, symbol 24LC512
- added U?: FT232R, symbol FT232R
- added U?: ENC28J60-I/SO, SOIC-28, symbol ENC28J60-I/SO
- added U? (x3): MCP23S17, symbol MCP23S17
Connections:
- net GND is gone; now on net +3V3: J?.1 (P1), J?.3 (P3)
- net +3V3: now also C?.1, C?.1, C?.1, C?.1, C?.2, C?.2, C?.2, C?.2, Q?.2 (E), R?.1, R?.1, R?.2, U?.1 (A0), U?.15 (A0), U?.15 (A0), U?.15 (A0), U?.16 (A1), U?.16 (A1), U?.16 (A1), U?.17 (A2), U?.17 (A2), U?.17 (A2), U?.17 (VSS), U?.18 (GND), U?.18 (VDD), U?.2 (A1), U?.21 (GND), U?.25 (AGND), U?.27 (VSS), U?.3 (A2), U?.30 (VDD), U?.39 (VSS), U?.4 (GND), U?.4 (VCCIO), U?.40 (VDD), U?.5 (VSS), U?.6 (~BOE), U?.7 (GND), U?.7 (WP), U?.8 (VCC), U?.8 (VDD)
- net +5V: now also J?.2 (Pin_2), U?.20 (VCC)
- net A1: now also U?.4 (GPB3)
- net A10: now also U?.25 (GPA4)
- net A11: now also U?.26 (GPA5)
- net A12: now also U?.27 (GPA6)
- net A13: now also U?.28 (GPA7)
- net A14: now also U?.1 (GPB0)
- net A15: now also U?.2 (GPB1)
- net A16: now also U?.3 (GPB2)
- net A17: now also U?.4 (GPB3)
- net A18: now also U?.5 (GPB4)
- net A19: now also U?.6 (GPB5)
- net A2: now also U?.5 (GPB4)
- net A20: now also U?.7 (GPB6)
- net A21: now also U?.8 (GPB7)
- net A22: now also U?.21 (GPA0)
- net A23: now also U?.22 (GPA1)
- net A3: now also U?.6 (GPB5)
- net A4: now also U?.7 (GPB6)
- net A5: now also U?.8 (GPB7)
- net A6: now also U?.21 (GPA0)
- net A7: now also U?.22 (GPA1)
- net A8: now also U?.23 (GPA2)
- net A9: now also U?.24 (GPA3)
- net D0: now also U?.1 (GPB0)
- net D1: now also U?.2 (GPB1)
- net D10: now also U?.23 (GPA2)
- net D11: now also U?.24 (GPA3)
- net D12: now also U?.25 (GPA4)
- net D13: now also U?.26 (GPA5)
- net D14: now also U?.27 (GPA6)
- net D15: now also U?.28 (GPA7)
- net D2: now also U?.3 (GPB2)
- net D3: now also U?.4 (GPB3)
- net D4: now also U?.5 (GPB4)
- net D5: now also U?.6 (GPB5)
- net D6: now also U?.7 (GPB6)
- net D7: now also U?.8 (GPB7)
- net D8: now also U?.21 (GPA0)
- net D9: now also U?.22 (GPA1)
- net R/~W: now also U?.1 (GPB0)
- net ~BG: now also U?.24 (GPA3)
- net ~BR: now also U?.23 (GPA2)
- net ~LDS: now also U?.2 (GPB1)
- net ~UDS: now also U?.3 (GPB2)
- new net: J?.1 (VBUS), L?.1
- new net: J?.1 (Pin_1), L?.2
- new net: R?.2, U?.1 (TXD)
- new net: R?.2, U?.5 (RXD)
- new net: C?.1, Q?.1 (B), R?.1
- new net FT232_TO_P8X32: R?.1, U?.38 (P31)
- new net MISO: U?.14 (SO), U?.14 (SO), U?.14 (SO)
- new net MOSI: U?.13 (SI), U?.13 (SI), U?.13 (SI)
- new net P8X32_TO_FT232: R?.1, U?.37 (P30)
- new net SCK: U?.12 (SCK), U?.12 (SCK), U?.12 (SCK)
- new net SCL: R?.2, U?.35 (P28), U?.6 (SCL)
- new net SDA: R?.2, U?.36 (P29), U?.5 (SDA)
- new net ~DTR: C?.2, U?.2 (~DTR)
- new net ~ETHER_CS: U?.9 (~CS)
- new net ~FLASH_CS: U?.1 (~CE)
- new net ~PE_CS: U?.11 (~CS), U?.11 (~CS), U?.11 (~CS)
- new net ~RST: Q?.3 (C), U?.7 (~RES)
- no-connect marks 3 -> 9
Other:
- note added: "Reicht ein CS für alle drei Portexpander?"
- note added: "Transistorpins prüfen"
- moved on the sheet: J?

Commit message: weiter
Parts:
- removed U?: ENC28J60-I/SO, SOIC-28, symbol ENC28J60-I/SO
- added C? (x5): 100n, symbol C_Small
- added J?: DB15_FEMALE_HighDensity_MountingHoles, symbol DB15_FEMALE_HighDensity_MountingHoles
- added J?: CONN_01X03, symbol CONN_01X03
- added R?: 0R, symbol R_Small
- added U?: PS2_female, symbol PS2_female
- added U?: WIZ820IO, symbol WIZ820IO
Connections:
- net +3V3: now also J?.4 (VDD), U?.3 (~WP), U?.7 (~HOLD), U?.8 (VDD), U?.9 (VCC), U?.9 (VCC), U?.9 (VCC), C?.1, C?.1, C?.1, C?.1, C?.1, R?.2, U?.10 (+3V3), U?.11 (+3V3); no longer C?.2, C?.2, C?.2, C?.2, J?.1 (P1), J?.3 (P3), Q?.2 (E), R?.2, U?.1 (A0), U?.15 (A0), U?.15 (A0), U?.16 (A1), U?.16 (A1), U?.17 (A2), U?.17 (A2), U?.17 (A2), U?.17 (VSS), U?.18 (GND), U?.2 (A1), U?.21 (GND), U?.25 (AGND), U?.27 (VSS), U?.3 (A2), U?.39 (VSS), U?.4 (GND), U?.5 (VSS), U?.6 (~BOE), U?.7 (GND), U?.7 (WP)
- net B: now also J?.3
- net G: now also J?.2
- net HS: now also J?.13
- net MISO: now also J?.7 (DAT0), U?.2 (SO), U?.7 (MISO)
- net MOSI: now also J?.2 (CMD), U?.5 (SI), U?.3 (MOSI)
- net PS2_CLK: now also U?.5 (CLK)
- net PS2_DAT: now also U?.1 (Data)
- net R: now also J?.1
- net SCK: now also J?.5 (CLK), U?.6 (SCK), U?.4 (SCLK)
- net VS: now also J?.14
- net ~ETHER_CS: now also U?.5 (~CS)
- net ~SD_CS: now also J?.1 (CD/DAT3)
- net USB_DM: now reaches J?.2 (D-)
- net USB_DM: now also U?.16 (USBDM)
- net USB_DP: now reaches J?.3 (D+)
- net USB_DP: now also U?.15 (USBDP)
- net GND: now reaches J?.4 (GND)
- net GND: now also C?.2, C?.2, C?.2, C?.2, J?.1 (P1), J?.3 (P3), J?.3 (VSS), J?.5 (Shield), J?.6 (VSS), Q?.2 (E), R?.2, U?.1 (A0), U?.10 (GND), U?.10 (GND), U?.10 (GND), U?.15 (A0), U?.15 (A0), U?.16 (A1), U?.16 (A1), U?.17 (A2), U?.17 (A2), U?.17 (A2), U?.17 (VSS), U?.18 (GND), U?.2 (A1), U?.21 (GND), U?.25 (AGND), U?.27 (VSS), U?.3 (A2), U?.39 (VSS), U?.4 (GND), U?.4 (VSS), U?.5 (VSS), U?.6 (~BOE), U?.7 (GND), U?.7 (WP), C?.2, C?.2, C?.2, C?.2, C?.2, J?.10, J?.5, J?.6, J?.7, J?.8, J?.9, U?.1 (GND), U?.12 (GND), U?.2 (GND), U?.3 (GND), U?.9 (PWDN)
- net SD_DETECT: now reaches J?.10 (CARD_DETECT)
- net SD_DETECT: now also U?.28 (GPA7)
- net ~PE_RESET: now reaches U?.18 (~RESET)
- net ~PE_RESET: now also U?.18 (~RESET), U?.18 (~RESET)
- net at U?.25 (GPA4): now also J?.3 (P3)
- net at U?.26 (GPA5): now also J?.2 (P2)
- net at U?.27 (GPA6): now also J?.1 (P1)
- new net: R?.1, U?.4 (VCC)
- new net ~ETHER_INT: U?.6 (~INT)
- new net ~ETHER_RESET: U?.8 (~RESET)
- no-connect marks 9 -> 14
Other:
- note added: "TODO:\n- Pinnummern vom Transistor prüfen\n- Reicht ein CS für die Portexpander?"
- note removed: "Reicht ein CS für alle drei Portexpander?"
- note removed: "Transistorpins prüfen"
- moved on the sheet: U?

Commit message: weiter
Parts:
- removed C?: 10n, symbol C_Small
- removed C? (x3): 100n, symbol C_Small
- removed J?: CONN_01X03, symbol CONN_01X03
- removed Q?: Q_NPN_BEC, symbol Q_NPN_BEC
- removed R?: 33k, symbol R_Small
- removed R? (x2): 150, symbol R_Small
- removed U?: FT232R, symbol FT232R
- removed U? (x3): MCP23S17, symbol MCP23S17
- added C? (x5): 100n, symbol C_Small
- added J?: PROP PLUG, symbol CONN_01X04
- added U?: DSPIC30F6014A, symbol DSPIC30F6014A
- added U?: FT230X, symbol FT230X
Connections:
- net +3V3: now also C?.1, C?.1, C?.1, C?.2, C?.2, U?.12 (VDD), U?.25 (AVDD), U?.32 (VDD), U?.48 (VDD), U?.71 (VDD)
- net GND: now also C?.1, C?.1, C?.2, C?.2, C?.2, U?.11 (VSS), U?.26 (AVSS), U?.31 (VSS), U?.51 (VSS), U?.70 (VSS)
- net MISO: now also U?.44 (SDI1/RF7)
- net MOSI: now also U?.43 (SDO1/RF8)
- net SCK: now also U?.45 (SCK1/INT0/RF6)
- net FT232_TO_P8X32 renamed PROP_RX
- net P8X32_TO_FT232 renamed PROP_TX
- new net PGC: U?.19 (PGC/RB1)
- new net PGD: U?.20 (PGD/RB0)
- new net UART_RX: U?.42 (U1RX/RF2)
- new net UART_TX: U?.41 (U1TX/RF3)
- new net ~MCLR: U?.9 (~MCLR)
- no-connect marks 14 -> 8
Other:
- note removed: "TODO:\n- Pinnummern vom Transistor prüfen\n- Reicht ein CS für die Portexpander?"
- moved on the sheet: C?, J?, R?, U?

Commit message: - iack fehlt auf m68k - extboard mit dspic30f6014a - zusätzlich propeller für terminal
Parts:
- added C?: 100n, symbol C_Small
- added C? (x2): 1µ, symbol C_Small
- added J?: ISP, symbol CONN_01X05
- added R? (x2): 10k, symbol R_Small
- added R? (x2): 100R, symbol R_Small
- added R? (x6): R_Small, symbol R_Small
- added R?: 4k7, symbol R_Small
- added U?: 74HC138, symbol 74HC138
- added U?: LM1117-3.3, symbol LM1117-3.3
Connections:
- net +3V3: now also U?.3 (VCCIO), C?.1, C?.1, J?.2 (P2), R?.1, R?.1, R?.1, U?.16 (VCC), U?.2 (VO), U?.4 (VO), U?.6 (E3); no longer J?.4 (P4), R?.2
- net +5V: now also R?.2, U?.12 (VCC), C?.2, U?.3 (VI)
- net A1: now also U?.73 (C1TX/RF1), U?.9 (P8)
- net A10: now also U?.2 (T2CK/RC1)
- net A11: now also U?.3 (T3CK/RC2)
- net A12: now also U?.4 (T4CK/RC3)
- net A13: now also U?.5 (T5CK/RC4)
- net A14: now also U?.6 (SCK2/RG6)
- net A15: now also U?.7 (SDI2/RG7)
- net A16: now also U?.8 (SDO2/RG8)
- net A17: now also U?.10 (SS2/RG9)
- net A18: now also U?.13 (INT1/RA12)
- net A19: now also U?.14 (INT2/RA13)
- net A2: now also U?.10 (P9), U?.74 (C2TX/RG1)
- net A20: now also U?.15 (AN5/RB5)
- net A21: now also U?.16 (AN4/RB4)
- net A22: now also U?.17 (AN3/RB3)
- net A23: now also U?.18 (AN2/SS2/RB2)
- net A3: now also U?.11 (P10), U?.75 (C2RX/RG0)
- net A4: now also U?.76 (CN22/RA6)
- net A5: now also U?.77 (CN23/RA7)
- net A6: now also U?.78 (RG14)
- net A7: now also U?.79 (RG12)
- net A8: now also U?.80 (RG13)
- net A9: now also U?.1 (COFS/RG15)
- net B0: now also U?.24 (P21), R?.2
- net B1: now also U?.25 (P22), R?.2
- net CS0: now also U?.1 (A0)
- net CS1: now also U?.2 (A1)
- net CS2: now also U?.3 (A2)
- net CS3: now also U?.5 (E2)
- net D0: now also U?.40 (U2TX/CN18/RF5), U?.41 (P0)
- net D1: now also U?.39 (U2RX/CN17/RF4), U?.42 (P1)
- net D10: now also U?.28 (AN9/RB9)
- net D11: now also U?.27 (AN8/RB8)
- net D12: now also U?.24 (RA10)
- net D13: now also U?.23 (RA9)
- net D14: now also U?.22 (AN7/RB7)
- net D15: now also U?.21 (AN6/RB6)
- net D2: now also U?.38 (IC8/CN21/RD15), U?.43 (P2)
- net D3: now also U?.37 (IC7/CN20/RD14), U?.44 (P3)
- net D4: now also U?.1 (P4), U?.36 (AN15/CN12/RB15)
- net D5: now also U?.2 (P5), U?.35 (AN14/RB14)
- net D6: now also U?.3 (P6), U?.34 (AN13/RB13)
- net D7: now also U?.33 (AN12/RB12), U?.4 (P7)
- net D8: now also U?.30 (AN11/RB11)
- net D9: now also U?.29 (AN10/RB10)
- net G0: now also U?.22 (P19), R?.2
- net G1: now also U?.23 (P20), R?.2
- net GND: now also J?.1 (P1), U?.13 (GND), U?.5 (GND), C?.1, C?.2, C?.2, J?.3 (P3), U?.1 (GND/ADJ), U?.4 (E1), U?.8 (GND); no longer J?.5 (Shield)
- net HS: now also U?.16 (P15)
- net PGC: now also J?.5 (P5)
- net PGD: now also J?.4 (P4)
- net PROP_RX: now also J?.3 (P3)
- net PROP_TX: now also J?.4 (P4)
- net PS2_CLK: now also U?.33 (P26), R?.1; no longer U?.5 (CLK)
- net PS2_DAT: now also U?.34 (P27), R?.1; no longer U?.1 (Data)
- net R/~W: now also U?.13 (P12), U?.63 (OC4/RD3)
- net R0: now also U?.20 (P17), R?.2
- net R1: now also U?.21 (P18), R?.2
- net SD_DETECT: now also U?.54 (IC1/RD8)
- net UART_RX: now also U?.1 (TXD)
- net UART_TX: now also U?.4 (RXD)
- net USB_DM: now also U?.9 (USBDM)
- net USB_DP: now also U?.8 (USBDP)
- net VS: now also U?.19 (P16)
- net ~AVEC: now also U?.66 (CN13/RD4)
- net ~BG: now also U?.60 (CN0/RC14)
- net ~BR: now also U?.61 (OC2/RD1)
- net ~DTACK: now also U?.62 (OC3/RD2)
- net ~ETHER_CS: now also U?.47 (SCL/RG2)
- net ~ETHER_INT: now also U?.50 (OSC2/CLKO/RC15)
- net ~FLASH_CS: now also U?.46 (SDA/RG3)
- net ~IPL0: now also U?.72 (C1RX/RF0)
- net ~IPL1: now also U?.69 (CN16/RD7)
- net ~IPL2: now also U?.68 (CN15/RD6)
- net ~LDS: now also U?.14 (P13), U?.64 (IC5/RD12)
- net ~MCLR: now also J?.1 (P1), R?.2
- net ~RST: now also J?.2 (P2)
- net ~SD_CS: now also U?.53 (INT4/RA15)
- net ~UDS: now also U?.65 (CN19/RD13)
- net ~VT_CS: now reaches U?.12 (P11)
- net ~VT_CS: now also U?.12 (O3)
- net IACK: now reaches U?.15 (P14)
- net IACK: now also U?.59 (CN1/RC13)
- net ~PIC_CS: now reaches U?.52 (INT3/RA14)
- net ~PIC_CS: now also U?.11 (O4)
- net ~IPL3: now reaches U?.67 (CN14/RD5)
- net ~RTS: now reaches U?.2 (~RTS)
- net ~CTS: now reaches U?.6 (~CTS)
- net B: no longer names the net of J?.3
- net B: now also R?.1, R?.1
- net G: no longer names the net of J?.2
- net G: now also R?.1, R?.1
- net R: no longer names the net of J?.1
- net R: now also R?.1, R?.1
- new net: R?.2, R?.2, U?.1 (Data)
- new net: R?.2, R?.2, U?.5 (CLK)
- new net +3V3_MAIN: J?.4 (P4)
Other:
- note added: "DEV_NONE = 0\nDEV_EEPROM = 1\nDEV_RAM = 2\nDEV_VT = 3\nDEV_PIC = 4\nDEV_OTHER = 5"
- moved on the sheet: C?, U?
